File: hardware/PCB/PCB.kicad_sch (KiCad schematic)
At the start: 30 parts, among them IC1 TSS721ADR, J1 Conn_01x02_Pin, J2 USB_C_Receptacle_USB2.0_14P, SW1 SW_Push, SW2 SW_Push, U1 ESP32-C6-MINI-1, U3 MCP1700x-330xxTT

Commit message: Finished initial schematic and PCB
Parts:
- removed C4: C, symbol Device:C
- removed C8: 330uF, symbol Device:C_Polarized
- removed IC1: TSS721ADR, Package_SO:SOIC-16_3.9x9.9mm_P1.27mm, symbol SS721ADR:TSS721ADR
- removed R1, R2: 220, Resistor_SMD:R_0805_2012Metric, symbol Device:R
- added C10: 1µF, Capacitor_SMD:C_0805_2012Metric, symbol Device:C
- added D4: SS14, Diode_SMD:D_SMA, symbol Diode:SS14
- added F1: Polyfuse, Inductor_SMD:L_1206_3216Metric_Pad1.22x1.90mm_HandSolder, symbol Device:Polyfuse
- added L2: 10uH, CR54NP221KC, symbol CR54NP-100MC:CR54NP-100MC
- added Q1: BC807, Package_TO_SOT_SMD:SOT-23, symbol Transistor_BJT:BC807
- added Q2, Q3: BC817, Package_TO_SOT_SMD:SOT-23, symbol Transistor_BJT:BC817
- added R12: 39K, Resistor_SMD:R_0805_2012Metric, symbol Device:R
- added R13: 33K, Resistor_SMD:R_0805_2012Metric, symbol Device:R
- added R14: 220K, Resistor_SMD:R_0805_2012Metric, symbol Device:R
- added R15: 82, Resistor_SMD:R_0805_2012Metric, symbol Device:R
- added R16, R17: 1K, Resistor_SMD:R_0805_2012Metric, symbol Device:R
- added R19: 22K, Resistor_SMD:R_0805_2012Metric, symbol Device:R
- added R20: 3K3, Resistor_SMD:R_0805_2012Metric, symbol Device:R
- added U2: AP3015, Package_TO_SOT_SMD:SOT-23-5, symbol Regulator_Switching:AP3012
- C2: value 10µ -> 22µ
- C6: value C -> 4.7µF; footprint (none) -> Capacitor_SMD:C_0805_2012Metric
- C9: value C -> 10µF; footprint (none) -> Capacitor_SMD:C_0805_2012Metric
- J1: footprint Connector_PinSocket_2.54mm:PinSocket_1x02_P2.54mm_Vertical -> TerminalBlock:TerminalBlock_MaiXu_MX126-5.0-02P_1x02_P5.00mm
- R10: value 100 -> 1M
- R11: value 100 -> 37K
- U1: footprint RF_Module:ESP32-C6-MINI-1 -> PCM_Espressif:ESP32-C6-MINI-1U
Connections:
- net +5V: now also F1.2
- net GND: now also C6.2, C10.2, Q2.2 (E), Q3.2 (E), R15.2, R19.2, R20.2, U2.2 (GND); no longer R10.2
- net LED: now also U1.20 (IO15); no longer U1.27 (IO21)
- net MBUS-: now also J1.2 (Pin_2), Q1.3 (C), R14.2
- net UART1_RX: now also R17.1
- net UART1_TX: now also R16.1
- net +36V: now reaches R10.1
- net +36V: now also C9.1, J1.1 (Pin_1), C10.1, D4.1 (K), R12.1, R13.1, R14.1, U2.1 (SW)
- net at R11.1: now also R10.2, U2.3 (FB)
- net at C6.1: now also F1.1, L2.1, U2.4 (~{SHDN}), U2.5 (IN)
- new net: D4.2 (A), L2.2
- new net: Q3.3 (C), R13.2, R17.2, R20.1
- new net: Q2.1 (B), R16.2
- new net: Q1.2 (E), Q3.1 (B), R15.1
- new net: Q1.1 (B), Q2.3 (C), R12.2, R19.1
- no-connect marks 18 -> 13
Other:
- title: (none) -> ESP32 M-Bus Adapter
- moved on the sheet: C5, D1, D2, D3, J1, R5, R6, R7, R8, R9, SW1, SW2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

Commit message: WIP - Adding BOM
Parts:
- C1: Mouse_PN (none) -> 80-C0805C104J4RAUTO
- C10: footprint Capacitor_SMD:C_0805_2012Metric -> Capacitor_SMD:C_1206_3216Metric; Mouse_PN (none) -> 80-C1206C105J5RECTU
- C2: Mouse_PN (none) -> 80-C0805C226M8P7210
- C3, C5, C7: Mouse_PN (none) -> 80-C0805C105J4RACLR
- C6: footprint Capacitor_SMD:C_0805_2012Metric -> Capacitor_SMD:C_1206_3216Metric; Mouse_PN (none) -> 80-C1206C475K5P
- C9: footprint Capacitor_SMD:C_0805_2012Metric -> Capacitor_SMD:C_1206_3216Metric; Mouse_PN (none) -> 80-C2220C106J5RACTU
- D1, D2, D3: Mouse_PN (none) -> 630-HSMH-H170
- D4: Mouse_PN (none) -> 512-SS14
- F1: Mouse_PN (none) -> 576-1206L050YR
- J2: Mouse_PN (none) -> 640-USB4105-GF-A
- L2: Mouse_PN (none) -> 851-CR54NP-100MC
- R3, R4, R6, R7, R8: Mouse_PN (none) -> 667-ERA-6ARW512V
- SW1, SW2: Mouse_PN (none) -> 640-SWT0110020010SSA
- U1: Mouse_PN (none) -> 356-ESP32-C6MINI1UH4
- U2: Mouse_PN (none) -> 621-AP3015AKTR-G1
- U3: Mouse_PN (none) -> 579-MCP1700T3302E/TT

Commit message: Finish BOMed and made some pad size adjustments for higher voltage tracks
Parts:
- Q1: Mouse_PN (none) -> 583-BC807
- Q2, Q3: Mouse_PN (none) -> 583-BC817
- R10: Mouse_PN (none) -> 603-RT0805FRE131ML
- R11: Mouse_PN (none) -> 603-RT0805FRE0737K4L
- R12: Mouse_PN (none) -> 603-RT0805BRD0739K2L
- R13: Mouse_PN (none) -> 603-AT0805BRE0733KL
- R14: Mouse_PN (none) -> 667-ERA-6AEB224V
- R15: Mouse_PN (none) -> 603-RT0805BRD0782RL
- R16, R17: Mouse_PN (none) -> 603-AT0805BRD071KL
- R19: Mouse_PN (none) -> 603-RT0805DRD0722KL
- R20: Mouse_PN (none) -> 603-RT0805FRE133K3L
- R5, R9: Mouse_PN (none) -> 603-RT0805BRD0710KL

Commit message: Add debugging header
Parts:
- added J3: Conn_01x04_Pin, Connector_PinHeader_2.54mm:PinHeader_1x04_P2.54mm_Vertical, symbol Connector:Conn_01x04_Pin
Connections:
- net +3.3V: now also J3.4 (Pin_4)
- net GND: now also J3.1 (Pin_1)
- net UART0_RX: now also J3.3 (Pin_3)
- net UART0_TX: now also J3.2 (Pin_2)

Commit message: Update BOM to correct C9
Parts:
- C9: Mouse_PN 80-C2220C106J5RACTU -> 187-CL31A106MBHNNNE
- J1, J3: now left out of the parts list
Changed lines of the file:
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@@
 	(title_block
 		(title "ESP32 M-Bus Adapter")
+		(date "2026-07-10")
+		(rev "B")
 	)
 	(junction
@@
 		(property "Mouse_PN" "603-RT0805BRD0710KL"
 			(at 25.4 140.97 0)
+			(hide yes)
 			(show_name no)
 			(do_not_autoplace no)
@@
 		(property "Mouse_PN" "851-CR54NP-100MC"
 			(at 143.51 25.4 0)
+			(hide yes)
 			(show_name no)
 			(do_not_autoplace no)
@@
 		(property "Mouse_PN" "603-AT0805BRE0733KL"
 			(at 149.86 85.09 0)
+			(hide yes)
 			(show_name no)
 			(do_not_autoplace no)
@@
 		(property "Mouse_PN" "603-RT0805FRE133K3L"
 			(at 149.86 127 0)
+			(hide yes)
 			(show_name no)
 			(do_not_autoplace no)
@@
 		(property "Mouse_PN" "603-AT0805BRD071KL"
 			(at 110.49 114.3 0)
+			(hide yes)
 			(show_name no)
 			(do_not_autoplace no)
@@
 		(property "Mouse_PN" "603-AT0805BRD071KL"
 			(at 110.49 107.95 0)
+			(hide yes)
 			(show_name no)
 			(do_not_autoplace no)
@@
 		(property "Mouse_PN" "512-SS14"
 			(at 168.91 25.4 0)
+			(hide yes)
 			(show_name no)
 			(do_not_autoplace no)
@@
 		(property "Mouse_PN" "80-C0805C105J4RACLR"
 			(at 62.23 133.35 0)
+			(hide yes)
 			(show_name no)
 			(do_not_autoplace no)
@@
 		(body_style 1)
 		(exclude_from_sim no)
-		(in_bom yes)
+		(in_bom no)
 		(on_board yes)
 		(in_pos_files yes)
@@
 			)
 		)
+		(property "Manufacturer_PN" ""
+			(at 265.43 30.48 0)
+			(hide yes)
+			(show_name no)
+			(do_not_autoplace no)
+			(effects
+				(font
+					(size 1.27 1.27)
+				)
+			)
+		)
+		(property "Mouse_PN" ""
+			(at 265.43 30.48 0)
+			(show_name no)
+			(do_not_autoplace no)
+			(effects
+				(font
+					(size 1.27 1.27)
+				)
+			)
+		)
 		(pin "1"
 		)
@@
 		(property "Mouse_PN" "621-AP3015AKTR-G1"
 			(at 152.4 39.37 0)
+			(hide yes)
 			(show_name no)
 			(do_not_autoplace no)
@@
 		(property "Mouse_PN" "603-RT0805BRD0710KL"
 			(at 62.23 120.65 0)
+			(hide yes)
 			(show_name no)
 			(do_not_autoplace no)
@@
 		(property "Mouse_PN" "576-1206L050YR"
 			(at 120.65 25.4 0)
+			(hide yes)
 			(show_name no)
 			(do_not_autoplace no)
@@
 		(property "Mouse_PN" "583-BC817"
 			(at 163.83 119.38 0)
+			(hide yes)
 			(show_name no)
 			(do_not_autoplace no)
@@
 		(property "Mouse_PN" "603-RT0805BRD0739K2L"
 			(at 138.43 85.09 0)
+			(hide yes)
 			(show_name no)
 			(do_not_autoplace no)
@@
 		(property "Mouse_PN" "583-BC817"
 			(at 123.19 107.95 0)
+			(hide yes)
 			(show_name no)
 			(do_not_autoplace no)
@@
 		(body_style 1)
 		(exclude_from_sim no)
-		(in_bom yes)
+		(in_bom no)
 		(on_board yes)
 		(in_pos_files yes)
@@
 			)
 		)
-		(property "Mouse_PN" "80-C2220C106J5RACTU"
+		(property "Mouse_PN" "187-CL31A106MBHNNNE"
 			(at 193.04 40.64 0)
+			(hide yes)
 			(show_name no)
 			(do_not_autoplace no)
@@
 		(property "Mouse_PN" "583-BC807"
 			(at 175.26 101.6 0)
+			(hide yes)
 			(show_name no)
 			(do_not_autoplace no)
@@
 		(property "Mouse_PN" "603-RT0805BRD0782RL"
 			(at 177.8 125.73 0)
+			(hide yes)
 			(show_name no)
 			(do_not_autoplace no)
@@
 		(property "Mouse_PN" "80-C1206C475K5P"
 			(at 128.27 35.56 0)
+			(hide yes)
 			(show_name no)
 			(do_not_autoplace no)
@@
 		(property "Mouse_PN" "603-RT0805FRE0737K4L"
 			(at 180.34 49.53 0)
+			(hide yes)
 			(show_name no)
 			(do_not_autoplace no)
@@
 		(property "Mouse_PN" "80-C1206C105J5RECTU"
 			(at 205.74 40.64 0)
+			(hide yes)
 			(show_name no)
 			(do_not_autoplace no)
@@
 		(property "Mouse_PN" "603-RT0805FRE131ML"
 			(at 180.34 33.02 0)
+			(hide yes)
 			(show_name no)
 			(do_not_autoplace no)
@@
 		(property "Mouse_PN" "603-RT0805DRD0722KL"
 			(at 138.43 127 0)
+			(hide yes)
 			(show_name no)
 			(do_not_autoplace no)
@@
 		(property "Mouse_PN" "667-ERA-6AEB224V"
 			(at 177.8 88.9 0)
+			(hide yes)
 			(show_name no)
 			(do_not_autoplace no)

Commit message: Slight tweak as previous component was out of stock
Parts:
- C9: Mouse_PN 187-CL31A106MBHNNNE -> 581-12065D106MAT2A
Changed lines of the file:
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@@
 			)
 		)
-		(property "Mouse_PN" "187-CL31A106MBHNNNE"
+		(property "Mouse_PN" "581-12065D106MAT2A"
 			(at 193.04 40.64 0)
 			(hide yes)

Commit message: WIP First pass through revision C
Connections:
- net MBUS-: now also Q1.2 (E); no longer Q1.3 (C)
- net at Q3.1 (B), R15.1: now also Q1.3 (C); no longer Q1.2 (E)
Changed lines of the file:
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@@
 	(title_block
 		(title "ESP32 M-Bus Adapter")
-		(date "2026-07-10")
-		(rev "B")
+		(date "2026-07-11")
+		(rev "C")
 	)
 	(junction
@@
 		(lib_id "Transistor_BJT:BC807")
 		(at 175.26 101.6 0)
+		(mirror x)
 		(unit 1)
 		(body_style 1)
@@
 		(in_pos_files yes)
 		(dnp no)
-		(fields_autoplaced yes)
 		(property "Reference" "Q1"
-			(at 180.34 100.3299 0)
+			(at 180.34 102.8701 0)
 			(show_name no)
 			(do_not_autoplace no)
@@
 		)
 		(property "Value" "BC807"
-			(at 180.34 102.8699 0)
+			(at 180.34 100.3301 0)
 			(show_name no)
 			(do_not_autoplace no)
@@
 		)
 		(property "Footprint" "Package_TO_SOT_SMD:SOT-23"
-			(at 180.34 103.505 0)
+			(at 180.34 99.695 0)
 			(hide yes)
 			(show_name no)

Commit message: More tweaks to revision C
Connections:
- net +3.3V: no longer J3.4 (Pin_4)
- net +5V: now also J3.4 (Pin_4)
Changed lines of the file:
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@@
 	(title_block
 		(title "ESP32 M-Bus Adapter")
-		(date "2026-07-11")
+		(date "2026-07-14")
 		(rev "C")
 	)
@@
 	)
 	(symbol
-		(lib_id "power:+3.3V")
-		(at 231.14 46.99 0)
-		(unit 1)
-		(body_style 1)
-		(exclude_from_sim no)
-		(in_bom yes)
-		(on_board yes)
-		(in_pos_files yes)
-		(dnp no)
-		(property "Reference" "#PWR030"
-			(at 231.14 50.8 0)
-			(hide yes)
-			(show_name no)
-			(do_not_autoplace no)
-			(effects
-				(font
-					(size 1.27 1.27)
-				)
-			)
-		)
-		(property "Value" "+3.3V"
-			(at 231.648 41.402 0)
-			(show_name no)
-			(do_not_autoplace no)
-			(effects
-				(font
-					(size 1.27 1.27)
-				)
-			)
-		)
-		(property "Footprint" ""
-			(at 231.14 46.99 0)
-			(hide yes)
-			(show_name no)
-			(do_not_autoplace no)
-			(effects
-				(font
-					(size 1.27 1.27)
-				)
-			)
-		)
-		(property "Datasheet" ""
-			(at 231.14 46.99 0)
-			(hide yes)
-			(show_name no)
-			(do_not_autoplace no)
-			(effects
-				(font
-					(size 1.27 1.27)
-				)
-			)
-		)
-		(property "Description" "Power symbol creates a global label with name \"+3.3V\""
-			(at 231.14 46.99 0)
-			(hide yes)
-			(show_name no)
-			(do_not_autoplace no)
-			(effects
-				(font
-					(size 1.27 1.27)
-				)
-			)
-		)
-		(pin "1"
-		)
-		(instances
-			(project "PCB"
-				(path "/e5b6d9ca-6ac8-47c6-8108-189de6594cb9"
-					(reference "#PWR030")
-					(unit 1)
-				)
-			)
-		)
-	)
-	(symbol
 		(lib_id "power:+5V")
 		(at 124.46 158.75 0)
@@
 					(unit 1)
 				)
+			)
+		)
+	)
+	(symbol
+		(lib_id "power:+5V")
+		(at 231.14 46.99 0)
+		(unit 1)
+		(body_style 1)
+		(exclude_from_sim no)
+		(in_bom yes)
+		(on_board yes)
+		(in_pos_files yes)
+		(dnp no)
+		(fields_autoplaced yes)
+		(property "Reference" "#PWR030"
+			(at 231.14 50.8 0)
+			(hide yes)
+			(show_name no)
+			(do_not_autoplace no)
+			(effects
+				(font
+					(size 1.27 1.27)
+				)
+			)
+		)
+		(property "Value" "+5V"
+			(at 231.14 41.91 0)
+			(show_name no)
+			(do_not_autoplace no)
+			(effects
+				(font
+					(size 1.27 1.27)
+				)
+			)
+		)
+		(property "Footprint" ""
+			(at 231.14 46.99 0)
+			(hide yes)
+			(show_name no)
+			(do_not_autoplace no)
+			(effects
+				(font
+					(size 1.27 1.27)
+				)
+			)
+		)
+		(property "Datasheet" ""
+			(at 231.14 46.99 0)
+			(hide yes)
+			(show_name no)
+			(do_not_autoplace no)
+			(effects
+				(font
+					(size 1.27 1.27)
+				)
+			)
+		)
+		(property "Description" "Power symbol creates a global label with name \"+5V\""
+			(at 231.14 46.99 0)
+			(hide yes)
+			(show_name no)
+			(do_not_autoplace no)
+			(effects
+				(font
+					(size 1.27 1.27)
+				)
+			)
+		)
+		(pin "1"
+		)
+		(instances
+			(project "PCB"
+				(path "/e5b6d9ca-6ac8-47c6-8108-189de6594cb9"
+					(reference "#PWR030")
+					(unit 1)
+				)
