File: hardware/PCB/PCB.kicad_sch (KiCad schematic)
At the start: 42 parts, among them J1 Conn_01x02_Pin, J2 USB_C_Receptacle_USB2.0_14P, J3 Conn_01x04_Pin, Q1 BC807, Q2 BC817, Q3 BC817, SW1 SW_Push, SW2 SW_Push, U1 ESP32-C6-MINI-1, U2 AP3015, U3 MCP1700x-330xxTT

Commit message: WIP
Connections:
- net +36V: no longer U2.1 (SW)
- net at D4.2 (A), L2.2: now also U2.1 (SW)
Other:
- moved on the sheet: C1, C2, D4, U1

Commit message: Revision F appears done.
I moved the capacitors and inductor positions.
Changed lines of the file:
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@@
 		(property "Mouse_PN" "640-USB4105-GF-A"
 			(at 227.33 106.68 0)
+			(hide yes)
 			(show_name no)
 			(do_not_autoplace no)

Commit message: Another few tweaks to tighten voltage booster components. Swapped debug header to remove long 5V trace
Connections:
- net UART0_RX: now also J3.2 (Pin_2); no longer J3.3 (Pin_3)
- net UART0_TX: now also J3.3 (Pin_3); no longer J3.2 (Pin_2)

Commit message: Small part number tweaks.
Parts:
- C10: Mouse_PN 80-C1206C105J5RECTU -> 963-MSASU319HB5105KT
- C2: Mouse_PN 80-C0805C226M8P7210 -> 963-MSASL21GBB5226MT
- C9: Mouse_PN 581-12065D106MAT2A -> 963-MLASU31LBB5106MT
- L2: Mouse_PN 851-CR54NP-100MC -> 851-CDRH5D18NP-100NC
- Q2, Q3: Mouse_PN 583-BC817 -> 637-BC817-25
Changed lines of the file:
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@@
 			)
 		)
-		(property "Mouse_PN" "851-CR54NP-100MC"
+		(property "Mouse_PN" "851-CDRH5D18NP-100NC"
 			(at 143.51 25.4 0)
 			(hide yes)
@@
 			)
 		)
-		(property "Mouse_PN" "80-C0805C226M8P7210"
+		(property "Mouse_PN" "963-MSASL21GBB5226MT"
 			(at 24.13 29.21 0)
 			(hide yes)
@@
 			)
 		)
-		(property "Mouse_PN" "583-BC817"
+		(property "Mouse_PN" "637-BC817-25"
 			(at 163.83 119.38 0)
 			(hide yes)
@@
 			)
 		)
-		(property "Mouse_PN" "583-BC817"
+		(property "Mouse_PN" "637-BC817-25"
 			(at 123.19 107.95 0)
 			(hide yes)
@@
 			)
 		)
-		(property "Mouse_PN" "581-12065D106MAT2A"
+		(property "Mouse_PN" "963-MLASU31LBB5106MT"
 			(at 193.04 40.64 0)
 			(hide yes)
@@
 			)
 		)
-		(property "Mouse_PN" "80-C1206C105J5RECTU"
+		(property "Mouse_PN" "963-MSASU319HB5105KT"
 			(at 205.74 40.64 0)
 			(hide yes)
