File: hardware/PCB/PCB.kicad_pcb (KiCad board)
At the start: 2 copper layers, 29.6 x 50.8 mm, 42 parts, among them J1 Conn_01x02_Pin, J2 USB_C_Receptacle_USB2.0_14P, J3 Conn_01x04_Pin, Q1 BC807, Q2 BC817, Q3 BC817, SW1 SW_Push, SW2 SW_Push, U1 ESP32-C6-MINI-1, U2 AP3015, U3 MCP1700x-330xxTT

Commit message: WIP First pass through revision C
Parts:
- moved R15 27.9 mm to (132.8, 60.7)
- moved Q3 27.3 mm to (133.9, 65.8), turned to 0 degrees
- moved C6 26.0 mm to (158.5, 55.9)
- moved C10 26.0 mm to (159.3, 42.4), turned to -90 degrees
- moved L2 22.8 mm to (154.7, 49.5), turned to -90 degrees
- moved C9 22.5 mm to (156.5, 42.4)
- moved R16 22.0 mm to (136.9, 58.2), turned to 90 degrees
- moved R17 21.9 mm to (136.9, 62.0), turned to -90 degrees
- moved R20 20.7 mm to (137.7, 66.8), turned to -90 degrees
- moved Q1 19.6 mm to (133.3, 53.3), turned to -90 degrees
- moved J3 19.1 mm to (158.2, 61.5), turned to 0 degrees
- moved F1 17.4 mm to (150.6, 56.1), turned to 180 degrees
- moved R13 16.9 mm to (143.5, 48.8), turned to -90 degrees
- moved R19 16.6 mm to (137.2, 50.0)
- moved R10 16.2 mm to (149.1, 40.9), turned to -90 degrees
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Connections:
- Q1 pad 2: Net-(Q1-E) -> MBUS-
- Q1 pad 3: MBUS- -> Net-(Q1-C)
- Q3 pad 1: Net-(Q1-E) -> Net-(Q1-C)
- R15 pad 1: Net-(Q1-E) -> Net-(Q1-C)
Routing:
- net GND: track 135.0 -> 81.6 mm, vias 9 -> 28
- net +3.3V: track 64.8 -> 40.1 mm, vias 3 -> 2
- net UART0_RX: track 24.7 -> 4.09 mm, vias 1 -> 0
- net UART0_TX: track 24.2 -> 4.27 mm, vias 1 -> 0
- net UART1_TX: track 2.80 -> 21.3 mm, vias 0 -> 2
- net UART1_RX: track 2.95 -> 21.4 mm, vias 0 -> 2
- net +5V: track 24.2 -> 42.3 mm
- net Net-(Q1-C): track 0.00 -> 11.1 mm
- net MBUS+: track 48.9 -> 38.5 mm
- net Net-(Q1-E): track 10.2 -> 0.00 mm
- net Net-(Q2-B): track 11.2 -> 2.55 mm, vias 2 -> 0
- net Net-(U2-IN): track 27.1 -> 20.4 mm, vias 4 -> 0
- net MBUS-: track 18.9 -> 12.5 mm
- net Net-(Q3-C): track 16.1 -> 22.5 mm
- net Net-(U2-FB): track 7.28 -> 4.86 mm
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Other:
- board size 29.6 x 50.8 mm -> 30.4 x 52.6 mm
- board text added: "M-"
- board text added: "Tomas McGuinness MBus-ESP32 Revision: ${REVISION}"

Commit message: WIP Revision C
Routing:
- net BOOT: track 16.5 -> 19.7 mm, vias 2 -> 0
- net GPIO8: track 9.65 -> 7.03 mm
- net UART1_RX: track 21.4 -> 23.3 mm
- net UART1_TX: track 21.3 -> 22.5 mm
- net +3.3V: track 40.1 -> 39.4 mm, vias 2 -> 0

Commit message: WIP track sizes
Routing:
- net EN: track 21.9 -> 24.6 mm
- net UART1_RX: track 23.3 -> 24.0 mm
- net GND: track 81.1 -> 81.8 mm

Commit message: More tweaks to revision C
Parts:
- moved R4 10.7 mm to (145.5, 77.7), turned to 90 degrees
- moved R5 1.19 mm to (135.4, 79.0), turned to 0 degrees
- moved C3 0.56 mm to (138.7, 76.2), turned to -90 degrees
- moved J3 0.51 mm to (158.8, 61.5)
Connections:
- J3 pad 4: +3.3V -> +5V
Routing:
- net +5V: track 42.3 -> 70.9 mm
- net Net-(J2-CC1): track 7.52 -> 4.98 mm
- net GND: track 81.8 -> 80.6 mm, vias 28 -> 29
Other:
- board text added: "5V"

Commit message: Added Front GND pour.
Routing:
- net GND: track 80.6 -> 23.5 mm, vias 29 -> 45
- net EN: track 24.4 -> 25.0 mm
- added copper zone on F.Cu, net GND

Commit message: Revision E!
Moved the two decoupling capacitors
Parts:
- moved C1 10.8 mm to (140.0, 66.0), turned to 180 degrees
- moved C2 7.23 mm to (140.0, 68.6), turned to 180 degrees
- moved R20 4.17 mm to (135.1, 70.1)
- moved R5 3.19 mm to (133.9, 76.2), turned to -90 degrees
Routing:
- net +3.3V: track 39.5 -> 34.5 mm
- net +5V: track 70.9 -> 72.3 mm
- net Net-(Q3-C): track 22.2 -> 23.3 mm
- net GND: track 23.5 -> 22.8 mm, vias 45 -> 40
