File: hardware/MBus-ESP-Adapter.kicad_sch (KiCad schematic)
At the start: 42 parts, among them J1 Conn_01x02_Pin, J2 USB_C_Receptacle_USB2.0_14P, J3 Conn_01x04_Pin, Q1 BC807, Q2 BC817, Q3 BC817, SW1 SW_Push, SW2 SW_Push, U1 ESP32-C6-MINI-1, U2 AP3015, U3 MCP1700x-330xxTT

Commit message: Fixed the USB footprint and symbol.
Parts:
- J2: value USB_C_Receptacle_USB2.0_14P -> USB_C_Receptacle_USB2.0_16P; symbol Connector:USB_C_Receptacle_USB2.0_14P -> Connector:USB_C_Receptacle_USB2.0_16P
Connections:
- net GND: now also J2.SH (SHIELD); no longer J2.S1 (SHIELD)
- no-connect marks 13 -> 16
