File: hardware/MBus-ESP-Adapter.kicad_sch (KiCad schematic)
At the start: 42 parts, among them J1 Conn_01x02_Pin, J2 USB_C_Receptacle_USB2.0_14P, J3 Conn_01x04_Pin, Q1 BC807, Q2 BC817, Q3 BC817, SW1 SW_Push, SW2 SW_Push, U1 ESP32-C6-MINI-1, U2 AP3015, U3 MCP1700x-330xxTT

Commit message: Start of Revision G
Parts:
- removed U3: MCP1700x-330xxTT, Package_TO_SOT_SMD:SOT-23, symbol Regulator_Linear:MCP1700x-330xxTT
- added U4: AP2112K-3.3, Package_TO_SOT_SMD:SOT-23-5, symbol Regulator_Linear:AP2112K-3.3
Connections:
- net +3.3V: now also U4.5 (VOUT)
- net +5V: now also U4.1 (VIN), U4.3 (EN)
- net GND: now also U4.2 (GND)

Commit message: Revision G tweaks
Parts:
- J2: symbol Connector:USB_C_Receptacle_USB2.0_14P -> Connector:USB_C_Receptacle_USB2.0_16P
Connections:
- net GND: now also J2.SH (SHIELD); no longer J2.S1 (SHIELD)
- no-connect marks 13 -> 15
Changed lines of the file:
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@@
 	)
 	(no_connect
+		(at 242.57 121.92)
+	)
+	(no_connect
 		(at 55.88 50.8)
 	)
@@
 	)
 	(no_connect
+		(at 242.57 119.38)
+	)
+	(no_connect
 		(at 86.36 66.04)
 	)
@@
 	)
 	(symbol
-		(lib_id "Connector:USB_C_Receptacle_USB2.0_14P")
+		(lib_id "Connector:USB_C_Receptacle_USB2.0_16P")
 		(at 227.33 106.68 0)
 		(unit 1)
@@
 			)
 		)
-		(property "Description" "USB 2.0-only 14P Type-C Receptacle connector"
+		(property "Description" "USB 2.0-only 16P Type-C Receptacle connector"
 			(at 227.33 106.68 0)
 			(hide yes)
@@
 			)
 		)
-		(pin "S1"
+		(pin "SH"
 		)
 		(pin "B1"
@@
 		(pin "B6"
 		)
+		(pin "B8"
+		)
+		(pin "A8"
+		)
 		(instances
