File: hardware/MBus-ESP-Adapter.kicad_pcb (KiCad board)
At the start: 2 copper layers, 30.4 x 52.6 mm, 42 parts, among them J1 Conn_01x02_Pin, J2 USB_C_Receptacle_USB2.0_14P, J3 Conn_01x04_Pin, Q1 BC807, Q2 BC817, Q3 BC817, SW1 SW_Push, SW2 SW_Push, U1 ESP32-C6-MINI-1, U2 AP3015, U3 MCP1700x-330xxTT

Commit message: Fixed the USB footprint and symbol.
Routing:
- net USB_D-: track 14.8 -> 15.9 mm
Changed lines of the file:
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@@
 	(title_block
 		(title "ESP32 M-Bus Adapter")
-		(date "2026-07-23")
-		(rev "F")
+		(date "2026-08-03")
+		(rev "G")
 		(comment 4 "AISLER Project ID: XWNAIXGJ")
 	)
@@
 		(capping no)
 		(filling no)
+		(zone_defaults)
 		(pcbplotparams
 			(layerselection 0x00000000_00000000_55555555_5755f5ff)
@@
 	)
 	(segment
-		(start 98.119 78.814529)
-		(end 97.818997 78.514526)
+		(start 98.119 80.798)
+		(end 98.119 78.814529)
 		(width 0.2)
 		(layer "F.Cu")
@@
 	)
 	(segment
-		(start 98.119 80.161)
-		(end 98.119 78.814529)
+		(start 99.393999 68.320999)
+		(end 99.393999 69.546001)
 		(width 0.2)
 		(layer "F.Cu")
@@
 	)
 	(segment
-		(start 99.393999 68.320999)
-		(end 99.393999 69.546001)
+		(start 98.119 80.19059)
+		(end 97.85141 79.923)
 		(width 0.2)
 		(layer "F.Cu")
@@
 	)
 	(segment
-		(start 97.119 79.165997)
-		(end 97.119 80.161)
+		(start 98.119 78.814529)
+		(end 97.818997 78.514526)
 		(width 0.2)
 		(layer "F.Cu")
@@
 	)
 	(segment
-		(start 97.818997 78.466)
-		(end 97.119 79.165997)
+		(start 98.119 80.798)
+		(end 98.119 80.19059)
+		(width 0.2)
+		(layer "F.Cu")
+		(net "USB_D-")
+	)
+	(segment
+		(start 97.85141 79.923)
+		(end 97.38659 79.923)
+		(width 0.2)
+		(layer "F.Cu")
+		(net "USB_D-")
+	)
+	(segment
+		(start 97.38659 79.923)
+		(end 97.119 80.19059)
 		(width 0.2)
 		(layer "F.Cu")
@@
 		(width 0.2)
 		(layer "F.Cu")
+		(net "USB_D-")
+	)
+	(segment
+		(start 97.119 80.19059)
+		(end 97.119 80.798)
+		(width 0.2)
+		(layer "F.Cu")

Commit message: Small tweak
Routing:
- net GND: track 23.1 -> 21.4 mm
Changed lines of the file:
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@@
 		(capping no)
 		(filling no)
-		(zone_defaults)
 		(pcbplotparams
 			(layerselection 0x00000000_00000000_55555555_5755f5ff)
@@
 		(layer "F.Cu")
 		(net "GND")
-	)
-	(segment
-		(start 94.069 58.296)
-		(end 94.069 59.996)
-		(width 0.2)
-		(layer "F.Cu")
-		(net "GND")
