File: hardware/MBus-ESP-Adapter.kicad_pcb (KiCad board)
At the start: 2 copper layers, 30.4 x 52.6 mm, 42 parts, among them J1 Conn_01x02_Pin, J2 USB_C_Receptacle_USB2.0_14P, J3 Conn_01x04_Pin, Q1 BC807, Q2 BC817, Q3 BC817, SW1 SW_Push, SW2 SW_Push, U1 ESP32-C6-MINI-1, U2 AP3015, U3 MCP1700x-330xxTT

Commit message: Start of Revision G
Parts:
- removed U3: MCP1700x-330xxTT, Package_TO_SOT_SMD:SOT-23
- added U4: AP2112K-3.3, Package_TO_SOT_SMD:SOT-23-5, F.Cu at (93.7, 74.2)
- moved C7 1.65 mm to (90.9, 78.5)
Routing:
- net +5V: track 62.6 -> 69.7 mm
- net +3.3V: track 34.5 -> 35.1 mm

Commit message: Revision G tweaks
Connections:
- J2 pad A8: (no net) -> unconnected-(J2-SBU1-PadA8)
- J2 pad B8: (no net) -> unconnected-(J2-SBU2-PadB8)
Routing:
- net +3.3V: track 35.1 -> 33.8 mm
- net +5V: track 69.7 -> 70.9 mm
Changed lines of the file:
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@@
 	(title_block
 		(title "ESP32 M-Bus Adapter")
-		(date "2026-07-23")
-		(rev "F")
+		(date "2026-09-02")
+		(rev "G")
 		(comment 4 "AISLER Project ID: XWNAIXGJ")
 	)
@@
 		(capping no)
 		(filling no)
+		(zone_defaults)
 		(pcbplotparams
 			(layerselection 0x00000000_00000000_55555555_5755f5ff)
@@
 			)
 		)
-		(property "Description" "USB 2.0-only 14P Type-C Receptacle connector"
+		(property "Description" "USB 2.0-only 16P Type-C Receptacle connector"
 			(at 0 0 0)
 			(unlocked yes)
@@
 			(unit
 				(name "A")
-				(pins "S1" "A1" "A12" "B1" "B12" "A4" "A9" "B4" "B9" "A5" "B5" "A7" "B7"
-					"A6" "B6"
+				(pins "SH" "A1" "A12" "B1" "B12" "A4" "A9" "B4" "B9" "A5" "B5" "A7" "B7"
+					"A6" "B6" "A8" "B8"
 				)
 			)
@@
 			(layers "F.Cu" "F.Mask" "F.Paste")
 			(roundrect_rratio 0.25)
+			(net "unconnected-(J2-SBU1-PadA8)")
+			(pinfunction "SBU1_A8")
+			(pintype "bidirectional+no_connect")
 		)
 		(pad "A9" smd roundrect
@@
 			(layers "F.Cu" "F.Mask" "F.Paste")
 			(roundrect_rratio 0.25)
+			(net "unconnected-(J2-SBU2-PadB8)")
+			(pinfunction "SBU2_B8")
+			(pintype "bidirectional+no_connect")
 		)
 		(pad "B9" smd roundrect
@@
 			(remove_unused_layers no)
 			(net "GND")
+			(pinfunction "SHIELD_SH")
+			(pintype "passive")
 		)
 		(pad "SH" thru_hole oval
@@
 			(remove_unused_layers no)
 			(net "GND")
+			(pinfunction "SHIELD_SH")
+			(pintype "passive")
 		)
 		(pad "SH" thru_hole oval
@@
 			(remove_unused_layers no)
 			(net "GND")
+			(pinfunction "SHIELD_SH")
+			(pintype "passive")
 		)
 		(pad "SH" thru_hole oval
@@
 			(remove_unused_layers no)
 			(net "GND")
+			(pinfunction "SHIELD_SH")
+			(pintype "passive")
 		)
 		(embedded_fonts no)
@@
 	)
 	(segment
-		(start 92.776 73.4715)
-		(end 92.776 73.0305)
-		(width 0.5)
-		(layer "F.Cu")
-		(net "+3.3V")
-	)
-	(segment
-		(start 93.319 60.846)
-		(end 94.119 60.846)
+		(start 92.469 61.696)
+		(end 93.319 60.846)
 		(width 0.5)
 		(layer "F.Cu")
@@
 	)
 	(segment
-		(start 92.579 71.5135)
-		(end 92.469 71.4035)
+		(start 90.437 72.606)
+		(end 90.475 72.644)
 		(width 0.5)
 		(layer "F.Cu")
@@
 	)
 	(segment
-		(start 92.469 71.6235)
-		(end 92.579 71.5135)
+		(start 90.475 72.644)
+		(end 92.3895 72.644)
 		(width 0.5)
 		(layer "F.Cu")
@@
 	)
 	(segment
-		(start 92.469 61.696)
-		(end 93.319 60.846)
+		(start 93.4805 70.612)
+		(end 92.469 69.6005)
 		(width 0.5)
 		(layer "F.Cu")
@@
 	)
 	(segment
-		(start 91.759 74.046)
-		(end 92.2015 74.046)
+		(start 92.469 71.4035)
+		(end 92.469 61.696)
 		(width 0.5)
 		(layer "F.Cu")
@@
 	)
 	(segment
-		(start 97.6205 72.286)
-		(end 101.694 72.286)
+		(start 93.319 60.846)
+		(end 94.119 60.846)
 		(width 0.5)
 		(layer "F.Cu")
@@
 	)
 	(segment
-		(start 92.2015 74.046)
-		(end 92.776 73.4715)
+		(start 92.3895 72.644)
+		(end 92.776 73.0305)
 		(width 0.5)
 		(layer "F.Cu")
@@
 	)
 	(segment
-		(start 90.437 72.724)
-		(end 91.759 74.046)
+		(start 97.6205 72.286)
+		(end 101.694 72.286)
 		(width 0.5)
 		(layer "F.Cu")
@@
 	)
 	(segment
-		(start 90.437 72.606)
-		(end 90.437 72.724)
-		(width 0.5)
-		(layer "F.Cu")
-		(net "+3.3V")
-	)
-	(segment
 		(start 85.357 72.6435)
 		(end 90.1455 72.6435)
@@
 	)
 	(segment
-		(start 92.776 73.0305)
-		(end 92.469 72.7235)
-		(width 0.5)
-		(layer "F.Cu")
-		(net "+3.3V")
-	)
-	(segment
-		(start 92.469 69.596)
-		(end 92.469 69.6005)
+		(start 92.776 71.7105)
+		(end 92.469 71.4035)
 		(width 0.5)
 		(layer "F.Cu")
@@
 	)
 	(segment
-		(start 92.469 72.7235)
-		(end 92.469 71.6235)
+		(start 92.776 73.0305)
+		(end 92.776 71.7105)
 		(width 0.5)
 		(layer "F.Cu")
@@
 	)
 	(segment
-		(start 92.469 69.6005)
-		(end 93.4805 70.612)
-		(width 0.5)
-		(layer "F.Cu")
-		(net "+3.3V")
-	)
-	(segment
 		(start 95.9465 70.612)
 		(end 96.3095 70.975)
@@
 	)
 	(segment
-		(start 92.469 71.4035)
-		(end 92.469 61.696)
-		(width 0.5)
-		(layer "F.Cu")
-		(net "+3.3V")
-	)
-	(segment
 		(start 85.357 74.4685)
 		(end 87.0315 74.4685)
@@
 	)
 	(via
-		(at 94.488 77.216)
+		(at 94.234 76.962)
 		(size 0.6)
 		(drill 0.3)
@@
 	)
 	(segment
-		(start 93.226001 74.193)
-		(end 94.259 74.193)
-		(width 0.5)
-		(layer "F.Cu")
-		(net "+5V")
-	)
-	(segment
 		(start 96.180001 82.084)
 		(end 95.469 81.372999)
@@
 	)
 	(segment
-		(start 92.776 74.643001)
-		(end 93.226001 74.193)
-		(width 0.5)
-		(layer "F.Cu")
-		(net "+5V")
-	)
-	(segment
 		(start 88.913 61.618)
 		(end 97.041 53.49)
@@
 	)
 	(segment
+		(start 95.469 76.0985)
+		(end 94.676 75.3055)
+		(width 0.5)
+		(layer "F.Cu")
+		(net "+5V")
+	)
+	(segment
 		(start 99.522695 82.084)
 		(end 96.180001 82.084)
@@
 	)
 	(segment
+		(start 95.469 79.813339)
+		(end 95.469 76.0985)
+		(width 0.5)
+		(layer "F.Cu")
+		(net "+5V")
+	)
+	(segment
 		(start 100.269 81.25541)
 		(end 100.269 80.798)
@@
 	)
 	(segment
-		(start 92.776 75.3055)
-		(end 92.776 74.643001)
-		(width 0.5)
-		(layer "F.Cu")
-		(net "+5V")
-	)
-	(segment
 		(start 91.882 78.486)
 		(end 94.141661 78.486)
@@
 	)
 	(segment
-		(start 94.676 74.61)
-		(end 94.676 75.3055)
-		(width 0.5)
-		(layer "F.Cu")
-		(net "+5V")
-	)
-	(segment
 		(start 88.913 69.238)
 		(end 88.913 61.618)
@@
 		(width 0.5)
 		(layer "F.Cu")
-		(net "+5V")
-	)
-	(segment
-		(start 94.259 74.193)
-		(end 94.676 74.61)
-		(width 0.5)
-		(layer "F.Cu")

Commit message: Revision G update
Other:
- board text added: "@tomasmcguinness MBus ESP32 Adapter Revision: ${REVISION}"
- board text added: "CA9M7"
- board text removed: "Tomás McGuinness MBus-ESP32 Revision: ${REVISION}"
Changed lines of the file:
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@@
+		)
+	)
+	(gr_text "CA9M7"
+		(at 82.55 73.914 270)
+		(layer "F.SilkS")
+		(effects
+			(font
+				(size 1 1)
+				(thickness 0.15)
+			)
+			(justify right bottom)
 		)
 	)
@@
 		)
 	)
-	(gr_text "Tomás McGuinness\nMBus-ESP32\nRevision: ${REVISION}"
+	(gr_text "@tomasmcguinness\nMBus ESP32 Adapter\nRevision: ${REVISION}"
 		(at 111.265 41.298 0)
 		(layer "B.SilkS")
